File: Project Architecture.kicad_sch (KiCad schematic)
At the start: 0 parts

Commit message: First draft of the schematic
Other:
- sheet Section A - Title A renamed Section A - Connectors
- sheet Section B - Title B renamed Section B - Arduino Mega
- added sheet Section C - LCL Selector (Section C - Title C.kicad_sch)
- note added: "Page 6"
