File: Section B - TItle B.kicad_sch (KiCad schematic)
At the start: 0 parts

Commit message: First draft of the schematic
Parts:
- added C3, C4, C5, C6, C7: 1uF, Capacitor_SMD:C_1206_3216Metric, symbol Device:C
- added DL1, DL2, DL3, DL4, DL5, DL6, DL7, T11, T12, T13, T15, T16, T17, T18, T19, T20, T21, T22, T23, T24, T25, T26, T27, T28, T29, T30, T31, T32, T33, T34, T35, T36, T37, T38, TTL1, TTL2, TTL3, TTL4, TTL5: TestPoint, TestPoint:TestPoint_Pad_1.0x1.0mm, symbol Connector:TestPoint
- added IC1: MAX232EIDR, SamacSys_Parts:SOIC127P600X175-16N, symbol SamacSys_Parts:MAX232EIDR
- added J1, J2, J3, J7, J8: 61300811121, Connector_PinHeader_2.54mm:PinHeader_1x08_P2.54mm_Vertical, symbol Connector_Generic:Conn_01x08
- added J4: 61304021121, Connector_PinHeader_2.54mm:PinHeader_2x18_P2.54mm_Vertical, symbol Connector_Generic:Conn_02x18_Odd_Even
- added J6: 61301211121, Connector_PinHeader_2.54mm:PinHeader_1x10_P2.54mm_Vertical, symbol Connector_Generic:Conn_01x10
- added J9: 61300811121, Connector_PinHeader_2.54mm:PinHeader_1x06_P2.54mm_Vertical, symbol Connector_Generic:Conn_01x06
- added Q13, Q22, Q4: IRLML2060, Package_TO_SOT_SMD:SOT-23, symbol Transistor_FET:IRLML2060
- added R1, R10, R2, R3, R4, R5, R56, R57, R6, R62, R7, R8, R9: 100R, Resistor_SMD:R_0805_2012Metric, symbol Device:R
- added R42, R43, R44: 100K, Resistor_SMD:R_0805_2012Metric, symbol Device:R
- added R66, R67, R68, R69, R70, R71, R72, R73, R74, R75: 10K, Resistor_SMD:R_0805_2012Metric, symbol Device:R
Connections:
- new net: J1.1 (Pin_1), T15.1
- new net: J7.5 (Pin_5), T11.1
- new net: J7.6 (Pin_6), T12.1
- new net: J4.10 (Pin_10), T33.1
- new net: J4.12 (Pin_12), T34.1
- new net: J4.14 (Pin_14), T35.1
- new net: J4.33 (Pin_33), T13.1
- new net: Q22.1 (G), R44.1, R62.2
- new net: C3.1, IC1.2 (VS+)
- new net: DL6.1, IC1.12 (ROUT1)
- new net: DL5.1, IC1.13 (RIN1)
- new net: Q4.1 (G), R43.1, R56.1
- new net: Q13.1 (G), R42.1, R57.1
- new net: C5.1, IC1.1 (C1+)
- new net: DL7.1, IC1.11 (DIN1)
- new net: DL4.1, IC1.14 (DOUT1)
- new net: C5.2, IC1.3 (C1-)
- new net: C6.1, IC1.4 (C2+)
- new net: C6.2, IC1.5 (C2-)
- new net: C4.1, IC1.6 (VS-)
- new net *10: J6.8 (Pin_8), R8.1
- new net *11: J6.7 (Pin_7), R7.1
- new net *12: J6.6 (Pin_6), R6.1
- new net *13: J6.5 (Pin_5), R5.1
- new net *4: J7.4 (Pin_4), R4.1
- new net *44: J4.11 (Pin_11), T27.1
- new net *46: J4.9 (Pin_9), T26.1
- new net *5: J7.3 (Pin_3), R3.1
- new net *6: J7.2 (Pin_2), R2.1
- new net *7: J7.1 (Pin_1), R1.1
- new net *8: J6.10 (Pin_10), R10.1
- new net *9: J6.9 (Pin_9), R9.1
- new net +3V3: J1.4 (Pin_4)
- new net +5V: C7.1, IC1.16 (VCC), J1.5 (Pin_5), J4.35 (Pin_35), J4.36 (Pin_36)
- new net 24: J4.31 (Pin_31), T32.1
- new net 26: J4.29 (Pin_29), T31.1
- new net 28: J4.27 (Pin_27), T30.1
- new net 32: J4.23 (Pin_23), T29.1
- new net 42: J4.13 (Pin_13), T28.1
- new net 48: J4.7 (Pin_7), T25.1
- new net 50: J4.5 (Pin_5), T24.1
- new net A0: J2.1 (Pin_1)
- new net A1: J2.2 (Pin_2)
- new net A10: J3.3 (Pin_3), T18.1
- new net A11: J3.4 (Pin_4), T19.1
- new net A12: J3.5 (Pin_5), T20.1
- new net A13: J3.6 (Pin_6), T21.1
- new net A14: J3.7 (Pin_7), T22.1
- new net A15: J3.8 (Pin_8), T23.1
- new net A2: J2.3 (Pin_3)
- new net A3: J2.4 (Pin_4)
- new net A4: J2.5 (Pin_5)
- new net A5: J2.6 (Pin_6)
- new net A6: J2.7 (Pin_7)
- new net A7: J2.8 (Pin_8)
- new net A8: J3.1 (Pin_1)
- new net A9: J3.2 (Pin_2)
- new net ARDU_UART_RX: IC1.9 (ROUT2), J8.2 (Pin_2)
- new net ARDU_UART_TX: IC1.10 (DIN2), J8.1 (Pin_1)
- new net AREF: J6.3 (Pin_3), T38.1
- new net DL1: DL1.1, J4.4 (Pin_4), R56.2
- new net DL2: DL2.1, J4.6 (Pin_6), R57.2
- new net DL3: DL3.1, J4.8 (Pin_8), R62.1
- new net DL_1_IN: Q4.3 (D)
- new net DL_1_OUT: Q4.2 (S), R43.2
- new net DL_2_IN: Q13.3 (D)
- new net DL_2_OUT: Q13.2 (S), R42.2
- new net DL_3_IN: Q22.3 (D)
- new net DL_3_OUT: Q22.2 (S), R44.2
- new net EL: J4.3 (Pin_3)
- new net GND: C3.2, C4.2, C7.2, IC1.15 (GND), J1.6 (Pin_6), J1.7 (Pin_7), J4.1 (Pin_1), J4.2 (Pin_2), J6.4 (Pin_4), R66.2, R67.2, R68.2, R69.2, R70.2, R71.2, R72.2, R73.2, R74.2, R75.2
- new net IOREF: J1.2 (Pin_2), T16.1
- new net K1: R4.2, R66.1
- new net K10: R5.2, R75.1
- new net K11: J4.15 (Pin_15)
- new net K12: J4.16 (Pin_16)
- new net K13: J4.17 (Pin_17)
- new net K14: J4.18 (Pin_18)
- new net K15: J4.19 (Pin_19)
- new net K16: J4.20 (Pin_20)
- new net K17: J4.21 (Pin_21)
- new net K18: J4.22 (Pin_22)
- new net K19: J4.25 (Pin_25)
- new net K2: R3.2, R67.1
- new net K20: J4.24 (Pin_24)
- new net K3: R2.2, R68.1
- new net K4: R1.2, R69.1
- new net K5: R10.2, R70.1
- new net K6: R71.1, R9.2
- new net K7: R72.1, R8.2
- new net K8: R7.2, R73.1
- new net K9: R6.2, R74.1
- new net RESET: J1.3 (Pin_3), T17.1
- new net RS232_RX_IN: IC1.8 (RIN2)
- new net RS232_TX_OUT: IC1.7 (DOUT2)
- new net RX0/0: J7.8 (Pin_8), T36.1
- new net RX1/19: J8.6 (Pin_6), J9.4 (Pin_4)
- new net RX2/17: J8.4 (Pin_4), J9.2 (Pin_2)
- new net SCL/21: J6.1 (Pin_1), J8.8 (Pin_8), J9.6 (Pin_6)
- new net SDA/20: J6.2 (Pin_2), J8.7 (Pin_7), J9.5 (Pin_5)
- new net TTL1: J4.30 (Pin_30), TTL1.1
- new net TTL2: J4.32 (Pin_32), TTL2.1
- new net TTL3: J4.28 (Pin_28), TTL3.1
- new net TTL4: J4.34 (Pin_34), TTL4.1
- new net TTL5: J4.26 (Pin_26), TTL5.1
- new net TX0/1: J7.7 (Pin_7), T37.1
- new net TX1/18: J8.5 (Pin_5), J9.3 (Pin_3)
- new net TX2/16: J8.3 (Pin_3), J9.1 (Pin_1)
- new net VCC: J1.8 (Pin_8)
Other:
- note added: "*2"
- note added: "*3"
- note added: "*44"
- note added: "*45"
- note added: "*46"
- note added: "*52"
- note added: "22"
- note added: "23"
- note added: "24"
- note added: "25"
- note added: "26"
- note added: "27"
- note added: "28"
- note added: "29"
- note added: "30"
- note added: "31"
- note added: "32"
- note added: "33"
- note added: "34"
- note added: "35"
- note added: "36"
- note added: "37"
- note added: "38"
- note added: "39"
- note added: "40"
- note added: "41"
- note added: "42"
- note added: "43"
- note added: "47"
- note added: "48"
- note added: "49"
- note added: "50"
- note added: "51"
- note added: "53"
- note added: "A0"
- note added: "A1"
- note added: "A2"
- note added: "A3"
- note added: "A4"
- note added: "A5"
- note added: "A6"
- note added: "A7"
- note added: "A8"
- note added: "A9"
- note added: "ANALOG"
- note added: "COMMUNICATION"
- note added: "DIGITAL"
- note added: "From PDCU"
- note added: "POWER"
- note added: "PWM"
- note added: "RX3/15"
- note added: "TX3/14"
- note added: "Vin"
- title: Sheet Title B -> Arduino Mega 2560
